Commit message: [fix]  add motors

File: pa10_description/urdf/pa10.xacro (robot description, xacro)
@@ -12,5 +12,5 @@
     <parent link="world"/>
     <child link="link0"/>
-    <origin rpy="0 0 0.523" xyz="0 0 .79"/>
+    <origin rpy="0 0 0" xyz="0 0 0"/>
   </joint>
   <link name="link0">
@@ -179,5 +179,5 @@
     <origin xyz="0 0 0.315" rpy="0 -0 0 "/>
     <axis   xyz="0 0 1"/>
-    <limit lower="-3.08923" upper="3.08923" effort="100000" velocity="0.4" />
+    <limit lower="-3.08923" upper="3.08923" effort="100000" velocity="50" />
     <dynamics damping="0.2" friction="0" />
   </joint>
@@ -187,5 +187,5 @@
     <origin xyz="0 0 0" rpy="0 -0 0 "/>
     <axis   xyz="0 1 0"/>
-    <limit lower="-1.58825" upper="1.58825" effort="100000" velocity="0.4" />
+    <limit lower="-1.58825" upper="1.58825" effort="100000" velocity="50" />
     <dynamics damping="0.2" friction="0" />
   </joint>
@@ -195,5 +195,5 @@
     <origin xyz="0 0 0" rpy="0 -0 0 "/>
     <axis   xyz="0 0 1"/>
-    <limit lower="-3.03687" upper="3.03687" effort="100000" velocity="0.5" />
+    <limit lower="-3.03687" upper="3.03687" effort="100000" velocity="50" />
     <dynamics damping="0.2" friction="0" />
   </joint>
@@ -203,5 +203,5 @@
     <origin xyz="0 0 0.450" rpy="0 -0 0 "/>
     <axis   xyz="0 1 0"/>
-    <limit lower="-2.3911" upper="2.3911" effort="100000" velocity="0.5" />
+    <limit lower="-2.3911" upper="2.3911" effort="100000" velocity="50" />
     <dynamics damping="0.2" friction="0" />
   </joint>
@@ -211,5 +211,5 @@
     <origin xyz="0 0 0" rpy="0 -0 0 "/>
     <axis   xyz="0 0 1"/>
-    <limit lower="-4.45059" upper="4.45059" effort="100000" velocity="0.5" />
+    <limit lower="-4.45059" upper="4.45059" effort="100000" velocity="50" />
     <dynamics damping="0.2" friction="0" />
   </joint>
@@ -219,5 +219,5 @@
     <origin xyz="0 0 0.5" rpy="0 -0 0 "/>
     <axis   xyz="0 1 0"/>
-    <limit lower="-2.87979" upper="2.87979" effort="100000" velocity="0.5" />
+    <limit lower="-2.87979" upper="2.87979" effort="100000" velocity="50" />
     <dynamics damping="0.2" friction="0" />
   </joint>
@@ -227,5 +227,5 @@
     <origin xyz="0 0 0.085" rpy="0 -0 0 "/>
     <axis   xyz="0 0 1"/>
-    <limit lower="-3.14159" upper="3.14159" effort="100000" velocity="0.5" />
+    <limit lower="-3.14159" upper="3.14159" effort="100000" velocity="50" />
     <dynamics damping="0.2" friction="0" />
     <!--<safety_controller k_position="100" k_velocity="1.5" soft_lower_limit="-2.857" soft_upper_limit="2.857"/>-->
@@ -235,3 +235,78 @@
       <origin xyz="0 0 0.02" rpy="0 0 0" />
   </xacro:schunk_pg70>
+  <transmission name="trans1">
+    <type>transmission_interface/SimpleTransmission</type>
+    <joint name="joint_1">
+      <hardwareInterface>PositionJointInterface</hardwareInterface>
+    </joint>
+    <actuator name="motor1">
+       <hardwareInterface>PositionJointInterface</hardwareInterface>
+      <mechanicalReduction>1</mechanicalReduction>
+    </actuator>
+  </transmission>
+  <transmission name="trans2">
+    <type>transmission_interface/SimpleTransmission</type>
+    <joint name="joint_2">
+      <hardwareInterface>PositionJointInterface</hardwareInterface>
+    </joint>
+    <actuator name="motor2">
+       <hardwareInterface>PositionJointInterface</hardwareInterface>
+      <mechanicalReduction>1</mechanicalReduction>
+    </actuator>
+  </transmission>
+  <transmission name="trans3">
+    <type>transmission_interface/SimpleTransmission</type>
+    <joint name="joint_3">
+      <hardwareInterface>PositionJointInterface</hardwareInterface>
+    </joint>
+    <actuator name="motor3">
+       <hardwareInterface>PositionJointInterface</hardwareInterface>
+      <mechanicalReduction>1</mechanicalReduction>
+    </actuator>
+  </transmission>
+  <transmission name="trans4">
+    <type>transmission_interface/SimpleTransmission</type>
+    <joint name="joint_4">
+      <hardwareInterface>PositionJointInterface</hardwareInterface>
+    </joint>
+    <actuator name="motor4">
+       <hardwareInterface>PositionJointInterface</hardwareInterface>
+      <mechanicalReduction>1</mechanicalReduction>
+    </actuator>
+  </transmission>
+  <transmission name="trans5">
+    <type>transmission_interface/SimpleTransmission</type>
+    <joint name="joint_5">
+      <hardwareInterface>PositionJointInterface</hardwareInterface>
+    </joint>
+    <actuator name="motor5">
+       <hardwareInterface>PositionJointInterface</hardwareInterface>
+      <mechanicalReduction>1</mechanicalReduction>
+    </actuator>
+  </transmission>
+  <transmission name="trans6">
+    <type>transmission_interface/SimpleTransmission</type>
+    <joint name="joint_6">
+      <hardwareInterface>PositionJointInterface</hardwareInterface>
+    </joint>
+    <actuator name="motor6">
+       <hardwareInterface>PositionJointInterface</hardwareInterface>
+      <mechanicalReduction>1</mechanicalReduction>
+    </actuator>
+  </transmission>
+  <transmission name="trans7">
+    <type>transmission_interface/SimpleTransmission</type>
+    <joint name="joint_7">
+      <hardwareInterface>PositionJointInterface</hardwareInterface>
+    </joint>
+    <actuator name="motor7">
+       <hardwareInterface>PositionJointInterface</hardwareInterface>
+      <mechanicalReduction>1</mechanicalReduction>
+    </actuator>
+  </transmission>
+  <gazebo>
+    <plugin name="gazebo_ros_control" filename="libgazebo_ros_control.so">
+      <robotNamespace>/pa10</robotNamespace>
+    </plugin>
+  </gazebo>
 </robot>
